File: bee-cab.sch (KiCad schematic (older format))
At the start: 24 parts, among them J1 Conn_01x02_Male, J10 Conn_01x01, J11 Conn_02x01, J12 Conn_02x01, J13 Conn_01x02, J14 Conn_01x02, J15 Conn_01x02, J16 Conn_01x02, J17 Conn_01x03, J2 Conn_01x02_Male, J3 Conn_01x02_Male, J4 Conn_01x02_Male, J5 Conn_01x03, J6 Conn_02x03_Odd_Even, J7 Conn_02x01, J8 Conn_01x02, J9 Conn_01x02

Commit message: Add pin sockets for custom parts.
Parts:
- added J18, J19: Conn_01x02, Connector_PinSocket_2.54mm:PinSocket_2x01_P2.54mm_Vertical, symbol Connector_Generic:Conn_01x02
Connections:
- net -15V: now also J19.1 (Pin_1), J19.2 (Pin_2)
- net at C1.2, C2.2, J17.1 (Pin_1)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: now also J18.1 (Pin_1), J18.2 (Pin_2)
Changed lines of the file:
@@
 Wire Wire Line
 	5250 4200 5250 3700
+$Comp
+L Connector_Generic:Conn_01x02 J18
+U 1 1 5CC336A4
+P 3950 4200
+F 0 "J18" H 4030 4192 50  0000 L CNN
+F 1 "Conn_01x02" H 4030 4101 50  0000 L CNN
+F 2 "Connector_PinSocket_2.54mm:PinSocket_2x01_P2.54mm_Vertical" H 3950 4200 50  0001 C CNN
+F 3 "~" H 3950 4200 50  0001 C CNN
+	1    3950 4200
+	1    0    0    -1
+$EndComp
+$Comp
+L Connector_Generic:Conn_01x02 J19
+U 1 1 5CC336AE
+P 3950 4500
+F 0 "J19" H 4030 4492 50  0000 L CNN
+F 1 "Conn_01x02" H 4030 4401 50  0000 L CNN
+F 2 "Connector_PinSocket_2.54mm:PinSocket_2x01_P2.54mm_Vertical" H 3950 4500 50  0001 C CNN
+F 3 "~" H 3950 4500 50  0001 C CNN
+	1    3950 4500
+	1    0    0    -1
+$EndComp
+Wire Wire Line
+	3750 4200 3750 4300
+Connection ~ 3750 4200
+Wire Wire Line
+	3750 4500 3750 4600
+Connection ~ 3750 4600
+Wire Wire Line
+	3750 4950 3500 4950
+Wire Wire Line
+	3750 4600 3750 4950
+Connection ~ 3500 4950
+Wire Wire Line
+	3750 3700 3500 3700
+Wire Wire Line
+	3750 3700 3750 4200
+Connection ~ 3500 3700
 $EndSCHEMATC
